File: Timebox_8/Aktiv ensretter/Active_rectifier.brd (EAGLE design)
At the start: 100 x 68.6 mm, 29 parts, among them Q1 BUZ10, Q2 BUZ10, Q3 BUZ10, Q4 BUZ10, Q5 BUZ10, Q6 BUZ10

Commit message: .sch og .brd filer ændret
Parts:
- added U$5, U$6, U$7, U$8: (no value), holes:3,0
- moved D2 1.27 mm to (85.1, 14.0)
- moved R1 1.27 mm to (85.1, 26.7)
- moved D5 1.27 mm to (58.4, 14.0)
- moved R3 1.27 mm to (58.4, 26.7)
Routing:
- net N$15: track 263.0 -> 379.5 mm
- net N$17: track 111.6 -> 225.6 mm
- net N$10: track 169.4 -> 255.8 mm
- net N$8: track 148.5 -> 219.8 mm
- net N$4: track 8.67 -> 9.94 mm
- net N$1: track 7.40 -> 8.39 mm
Other:
- board size 100 x 68.6 mm -> 108.9 x 68.6 mm
